Commit message: new moveit for scara

File: scara_moveit/config/gazebo_scara_mit_dh_urdf.urdf (robot description, URDF)
Before this commit: robot scara_mit_dh_urdf, 6 links, 5 joints
Links:
- removed link Gripper
- removed link joint_1
- removed link joint_2
- removed link joint_3
- removed link joint_4
- added link l1, mass 49.5926714803606; collision mesh filename=package://scara_mit_dh_urdf/meshes/l1.STL; visual mesh filename=package://scara_mit_dh_urdf/meshes/l1.STL
- added link l2, mass 32.5846948095504; collision mesh filename=package://scara_mit_dh_urdf/meshes/l2.STL; visual mesh filename=package://scara_mit_dh_urdf/meshes/l2.STL
- added link l3, mass 0.460306155603976; collision mesh filename=package://scara_mit_dh_urdf/meshes/l3.STL; visual mesh filename=package://scara_mit_dh_urdf/meshes/l3.STL
- added link l4, mass 0.00734707672394354; collision mesh filename=package://scara_mit_dh_urdf/meshes/l4.STL; visual mesh filename=package://scara_mit_dh_urdf/meshes/l4.STL
- added link world
- link base_link: mass 46.1322926928931 -> 50.5064528015554; geometry collision mesh filename=package://scara_mit_dh_urdf/meshes/base_link.STL; visual mesh filename=package://scara_mit_dh_urdf/meshes/base_link.STL
Joints:
- removed joint Saugnapf
- removed joint arm1
- removed joint arm2
- removed joint arm3
- removed joint arm4
- added joint fixedToWorld: type fixed, parent world, child base_link, origin xyz=0 0 1 rpy=0 0 0
- added joint j1: type revolute, parent base_link, child l1, origin xyz=0 -0.375 0 rpy=1.5708 0 0, axis 0 0 1, limit lower=-2.7 upper=2.7 effort=10000 velocity=1
- added joint j2: type revolute, parent l1, child l2, origin xyz=0.325 0 0.06 rpy=3.1416 0 3.1416, axis 0 0 1, limit lower=-2.7 upper=2.7 effort=10000 velocity=1
- added joint j3: type prismatic, parent l2, child l3, origin xyz=-0.225 0 0.06926 rpy=0 0 0, axis 0 0 1, limit lower=0 upper=290 effort=10000 velocity=1
- added joint j4: type revolute, parent l3, child l4, origin xyz=0 0 0 rpy=0 0 -3.0137, axis 0 0 1, limit lower=-6.2 upper=6.2 effort=10000 velocity=1
