Commit message: try on automatic

File: rod_moveit/config/gazebo_rod_projekt2.urdf (robot description, URDF)
Before this commit: robot rod_projekt2, 20 links, 19 joints
Joints:
- joint saj4: limit lower=-4 upper=4 effort=10 velocity=9.8 -> lower=-7 upper=7 effort=10 velocity=9.8
- joint saj6: limit lower=-7 upper=7 effort=10 velocity=13.1 -> lower=-14 upper=14 effort=100 velocity=13.1

File: rod_projekt2/urdf/rod_projekt2.urdf (robot description, URDF)
Before this commit: robot rod_projekt2, 20 links, 19 joints
Joints:
- joint saEE1: limit lower=-0.02 upper=0 effort=10 velocity=3.14 -> lower=-0.02 upper=0 effort=10000 velocity=3.14
- joint saEE2: limit lower=0 upper=0.02 effort=10 velocity=3.14 -> lower=0 upper=0.02 effort=10000 velocity=3.14
- joint saj1: limit lower=-4.3 upper=4.3 effort=10 velocity=8 -> lower=-4.3 upper=4.3 effort=10000 velocity=8
- joint saj2: limit lower=-2 upper=2 effort=10 velocity=6.6 -> lower=-2 upper=2 effort=10000 velocity=6.6
- joint saj3: limit lower=-3.6 upper=1 effort=10 velocity=4.9 -> lower=-3.6 upper=1 effort=10000 velocity=4.9
- joint saj4: limit lower=-4 upper=4 effort=10 velocity=9.8 -> lower=-7 upper=7 effort=10000 velocity=9.8
- joint saj5: limit lower=-2.2 upper=2.1 effort=10 velocity=7.3 -> lower=-2.2 upper=2.1 effort=10000 velocity=7.3
- joint saj6: limit lower=-7 upper=7 effort=10 velocity=13.1 -> lower=-14 upper=14 effort=10000 velocity=13.1
- joint sj1: limit lower=-2.7 upper=2.7 effort=10 velocity=9.2 -> lower=-2.7 upper=2.7 effort=10000 velocity=9.2
- joint sj2: limit lower=-2.7 upper=2.7 effort=10 velocity=9.2 -> lower=-2.7 upper=2.7 effort=10000 velocity=9.2
- joint sj3: limit lower=0 upper=0.32 effort=10 velocity=2 -> lower=0 upper=0.32 effort=10000 velocity=2
- joint sjEE: limit lower=-6.2 upper=6.2 effort=10 velocity=41.9 -> lower=-6.2 upper=6.2 effort=10000 velocity=41.9
