Commit message: moveit setup assistant correction

File: rod/urdf/rod.urdf (robot description, URDF)
Before this commit: robot rod, 23 links, 22 joints
Links:
- added link world
Joints:
- added joint fixed_link_to_world: type fixed, parent world, child base_link

Commit message: try on automation robots

File: rod/urdf/rod.urdf (robot description, URDF)
Before this commit: robot rod, 24 links, 23 joints
Joints:
- joint saj6: limit lower=-7 upper=7 effort=10 velocity=9.8 -> lower=-3.2 upper=3.2 effort=10 velocity=9.8

Commit message: new working automatic project

File: rod/urdf/rod.urdf (robot description, URDF)
Before this commit: robot rod, 24 links, 23 joints
Links:
- link sixaxis_j6: mass 1.14880650871049 -> 1.25901265956962
Joints:
- removed joint fixed_link_to_world
- added joint FixedLinkToWorld: type fixed, parent world, child base_link
- joint pj1: limit lower=-1.5 upper=0 effort=10 velocity=4 -> lower=-1.5 upper=0 effort=10000 velocity=4
- joint pj2: limit lower=-2.3 upper=2.3 effort=10 velocity=9 -> lower=-2.3 upper=2.3 effort=1000 velocity=9
- joint pj3: limit lower=-2.6 upper=2.6 effort=10 velocity=9 -> lower=-2.6 upper=2.6 effort=1000 velocity=9
- joint pj4: limit lower=-7 upper=7 effort=10 velocity=8.4 -> lower=-7 upper=7 effort=1000 velocity=8.4
- joint sEE: limit lower=-6.2 upper=6.2 effort=10 velocity=41.9 -> lower=-6.2 upper=6.2 effort=1000 velocity=41.9
- joint saj1: limit lower=-4.3 upper=4.3 effort=10 velocity=8 -> lower=-4.3 upper=4.3 effort=1000 velocity=8
- joint saj2: limit lower=-2 upper=2 effort=10 velocity=6.6 -> lower=-2 upper=2 effort=1000 velocity=6.6
- joint saj3: limit lower=-3.6 upper=1 effort=10 velocity=4.9 -> lower=-3.6 upper=1 effort=1000 velocity=4.9
- joint saj4: limit lower=-4 upper=4 effort=10 velocity=9.8 -> lower=-4 upper=4 effort=1000 velocity=9.8
- joint saj5: limit lower=-2.2 upper=2.1 effort=10 velocity=7.3 -> lower=-2.2 upper=2.1 effort=1000 velocity=7.3
- joint saj6: axis 0 0 1 -> 0 0 -1; limit lower=-3.2 upper=3.2 effort=10 velocity=9.8 -> lower=-7 upper=7 effort=1000 velocity=9.8; origin xyz=-0.027996 -0.12051 0 rpy=-1.5708 1.5535 -3.1416 -> xyz=0 -0.151 0 rpy=1.5708 0 0
- joint sj1: limit lower=-2.7 upper=2.7 effort=10 velocity=9.2 -> lower=-2.7 upper=2.7 effort=1000 velocity=9.2
- joint sj2: limit lower=-2.7 upper=2.7 effort=10 velocity=7.9 -> lower=-2.7 upper=2.7 effort=1000 velocity=7.9
- joint sj3: limit lower=0 upper=0.32 effort=10 velocity=2 -> lower=0 upper=0.32 effort=1000 velocity=2
